Commit message: add gazebo launch add controllers for manipulator changed position of camera

File: urdf/two_link_manipulator.xacro (robot description, xacro)
@@ -1,5 +1,5 @@
 <?xml version="1.0"?>
-<robot name="two_link_manipulator" xmlns:xacro="http://wiki.ros.org/xacro">
-    <xacro:property name="DEG2RAD" value="0.017453292519943295"/>
+<robot name="two_link_manipulator">
+    <property name="DEG2RAD" value="0.017453292519943295"/>
     <macro name="box_link" params="name xyz rpy size">
         <link name="${name}">
@@ -16,9 +16,9 @@
                 </geometry>
             </collision>
-            <inertia>
+            <inertial>
                 <origin xyz="${xyz}" rpy="${rpy}"/>
                 <mass value="1"/>
-                <inertia ixx="0" ixy="0" ixz="0" iyy="0" iyz="0" izz="0"/>
-            </inertia>
+                <inertia ixx="1.0" ixy="0.0" ixz="0.0" iyy="1.0" iyz="0.0" izz="1.0"/>
+            </inertial>
         </link>
     </macro>
@@ -30,11 +30,33 @@
             <axis xyz="${axis}"/>
             <limit effort="100" lower="${lower}" upper="${upper}" velocity="${vel}"/>
-            <dynamics damping="5" friction="10"/>
+            <dynamics damping="1" friction="1"/>
         </joint>
     </macro>
+    <macro name="joint_transmission" params="joint">
+        <transmission name="trans_${joint}">
+            <type>
+                transmission_interface/SimpleTransmission
+            </type>
+            <joint name="${joint}">
+                <hardwareInterface>
+                    hardware_interface/EffortJointInterface
+                </hardwareInterface>
+            </joint>
+            <actuator name="motor_${joint}">
+                <hardwareInterface>
+                    hardware_interface/EffortJointInterface
+                </hardwareInterface>
+                <mechanicalReduction>
+                    1
+                </mechanicalReduction>
+            </actuator>
+        </transmission>
+    </macro>
+    <!--LINKS-->
     <link name="world"/>
     <box_link name="base_link" xyz="0 0 0.5" rpy="0 0 0" size="0.2 0.2 1"/>
     <box_link name="link1" xyz="0 0 0.3" rpy="0 0 0" size="0.05 0.05 0.6"/>
     <box_link name="link2" xyz="0 0 0.1625" rpy="0 0 0" size="0.05 0.05 0.375"/>
+    <!--JOINTS-->
     <joint name="base_world" type="fixed">
         <origin xyz="0 0 0" rpy="0 0 0"/>
@@ -42,8 +64,20 @@
         <child link="base_link"/>
     </joint>
-    <revolute_joint name="joint1" xyz="0 0.125 0.95" rpy="0 ${DEG2RAD * 90} 0" parent="base_link" child="link1" axis="0 1 0"
+    <revolute_joint name="joint1" xyz="0 0.125 0.95" rpy="0 ${DEG2RAD * 90} 0" parent="base_link" child="link1"
+                    axis="0 1 0"
                     lower="${-DEG2RAD * 179.9}" upper="${DEG2RAD * 180}" vel="1"/>
     <revolute_joint name="joint2" xyz="0 0.05 0.575" rpy="0 0 0" parent="link1" child="link2" axis="0 1 0"
                     lower="${-DEG2RAD * 179.9}" upper="${DEG2RAD * 180}" vel="1"/>
+    <joint_transmission joint="joint1"/>
+    <joint_transmission joint="joint2"/>
+    <gazebo reference="base_link">
+        <material>Gazebo/White</material>
+    </gazebo>
+    <gazebo reference="link1">
+        <material>Gazebo/Orange</material>
+    </gazebo>
+    <gazebo reference="link2">
+        <material>Gazebo/White</material>
+    </gazebo>
     <gazebo>
         <plugin name="gazebo_ros_control" filename="libgazebo_ros_control.so"/>

Commit message: rviz changed control added

File: urdf/two_link_manipulator.xacro (robot description, xacro)
@@ -10,10 +10,10 @@
                 </geometry>
             </visual>
-            <collision>
+<!--             <collision>
                 <origin xyz="${xyz}" rpy="${rpy}"/>
                 <geometry>
                     <box size="${size}"/>
                 </geometry>
-            </collision>
+            </collision> -->
             <inertial>
                 <origin xyz="${xyz}" rpy="${rpy}"/>
@@ -55,28 +55,28 @@
     <!--LINKS-->
     <link name="world"/>
-    <box_link name="base_link" xyz="0 0 0.5" rpy="0 0 0" size="0.2 0.2 1"/>
-    <box_link name="link1" xyz="0 0 0.3" rpy="0 0 0" size="0.05 0.05 0.6"/>
-    <box_link name="link2" xyz="0 0 0.1625" rpy="0 0 0" size="0.05 0.05 0.375"/>
+    <box_link name="base_link" xyz="0.1 0.1 1.05" rpy="0 0 0" size="0.2 0.2 2.1"/>
+    <box_link name="link1" xyz="0.05 0.05 0.5" rpy="0 0 0" size="0.1 0.1 1.0"/>
+    <box_link name="link2" xyz="0.05 0.05 0.5" rpy="0 0 0" size="0.1 0.1 1.0"/>
     <!--JOINTS-->
     <joint name="base_world" type="fixed">
-        <origin xyz="0 0 0" rpy="0 0 0"/>
+        <origin xyz="-0.1 -0.1 0" rpy="0 0 0"/>
         <parent link="world"/>
         <child link="base_link"/>
     </joint>
-    <revolute_joint name="joint1" xyz="0 0.125 0.95" rpy="0 ${DEG2RAD * 90} 0" parent="base_link" child="link1"
+    <revolute_joint name="joint1" xyz="0 0.25 2.1" rpy="0 -${DEG2RAD * 90} 0" parent="base_link" child="link1"
                     axis="0 1 0"
                     lower="${-DEG2RAD * 179.9}" upper="${DEG2RAD * 180}" vel="1"/>
-    <revolute_joint name="joint2" xyz="0 0.05 0.575" rpy="0 0 0" parent="link1" child="link2" axis="0 1 0"
+    <revolute_joint name="joint2" xyz="0 0.1 1" rpy="0 0 0" parent="link1" child="link2" axis="0 1 0"
                     lower="${-DEG2RAD * 179.9}" upper="${DEG2RAD * 180}" vel="1"/>
     <joint_transmission joint="joint1"/>
     <joint_transmission joint="joint2"/>
     <gazebo reference="base_link">
-        <material>Gazebo/White</material>
+        <material>Gazebo/Black</material>
     </gazebo>
     <gazebo reference="link1">
-        <material>Gazebo/Orange</material>
+        <material>Gazebo/Red</material>
     </gazebo>
     <gazebo reference="link2">
-        <material>Gazebo/White</material>
+        <material>Gazebo/Green</material>
     </gazebo>
     <gazebo>
